File: electronics/kicad/robo-sumo.kicad_pcb (KiCad board)
At the start: 2 copper layers, 100 x 70 mm, 13 parts

Commit message: pcb: save unrouted board layout
Parts:
- moved J_PW1 1.05 mm to (105.2, 98.8)
- moved J_D1 1.02 mm to (122.5, 134.9)
- moved J_G1 1.02 mm to (141.1, 134.9)
- moved J_PW2 1.02 mm to (105.2, 107.7)
- moved J_D2 0.77 mm to (159.4, 74.9)
- moved J_L3 0.77 mm to (181.8, 74.9)
- moved J_P2 0.77 mm to (129.6, 74.9)
- moved J_P3 0.77 mm to (140.7, 74.9)
- moved J_P1 0.77 mm to (118.5, 74.9)
- moved J_L1 0.77 mm to (170.7, 74.9)
- moved J_L2 0.77 mm to (193.0, 74.9)
Routing:
- net /L_RPWM: track 13.1 -> 0.00 mm
- net /PROX_F_HV: track 2.16 -> 0.00 mm
- net /LINE_L: track 1.70 -> 0.00 mm
- net /LINE_B: track 0.92 -> 0.00 mm
- net +3.3V: track 0.61 -> 0.00 mm
- removed copper zone on B.Cu, net GND
Changed lines of the file:
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@@
 	(footprint "Connector_JST:JST_XH_B6B-XH-A_1x06_P2.50mm_Vertical"
 		(layer "F.Cu")
-		(at 122.368 135.89)
+		(at 122.461 134.874)
 		(descr "JST XH series connector, B6B-XH-A (http://www.jst-mfg.com/product/pdf/eng/eXH.pdf), generated with kicad-footprint-generator")
 		(tags "connector JST XH vertical")
@@
 	(footprint "Connector_JST:JST_XH_B4B-XH-A_1x04_P2.50mm_Vertical"
 		(layer "F.Cu")
-		(at 140.97 135.89)
+		(at 141.063 134.874)
 		(descr "JST XH series connector, B4B-XH-A (http://www.jst-mfg.com/product/pdf/eng/eXH.pdf), generated with kicad-footprint-generator")
 		(tags "connector JST XH vertical")
@@
 	(footprint "Connector_JST:JST_XH_B3B-XH-A_1x03_P2.50mm_Vertical"
 		(layer "F.Cu")
-		(at 118.618 74.168 180)
+		(at 118.491 74.93 180)
 		(descr "JST XH series connector, B3B-XH-A (http://www.jst-mfg.com/product/pdf/eng/eXH.pdf), generated with kicad-footprint-generator")
 		(tags "connector JST XH vertical")
@@
 	(footprint "Connector_JST:JST_XH_B3B-XH-A_1x03_P2.50mm_Vertical"
 		(layer "F.Cu")
-		(at 193.134 74.168 180)
+		(at 193.007 74.93 180)
 		(descr "JST XH series connector, B3B-XH-A (http://www.jst-mfg.com/product/pdf/eng/eXH.pdf), generated with kicad-footprint-generator")
 		(tags "connector JST XH vertical")
@@
 	(footprint "Connector_JST:JST_XH_B3B-XH-A_1x03_P2.50mm_Vertical"
 		(layer "F.Cu")
-		(at 140.81 74.168 180)
+		(at 140.683 74.93 180)
 		(descr "JST XH series connector, B3B-XH-A (http://www.jst-mfg.com/product/pdf/eng/eXH.pdf), generated with kicad-footprint-generator")
 		(tags "connector JST XH vertical")
@@
 	(footprint "Connector_JST:JST_XH_B3B-XH-A_1x03_P2.50mm_Vertical"
 		(layer "F.Cu")
-		(at 181.958 74.168 180)
+		(at 181.831 74.93 180)
 		(descr "JST XH series connector, B3B-XH-A (http://www.jst-mfg.com/product/pdf/eng/eXH.pdf), generated with kicad-footprint-generator")
 		(tags "connector JST XH vertical")
@@
 	(footprint "Connector_JST:JST_XH_B6B-XH-A_1x06_P2.50mm_Vertical"
 		(layer "F.Cu")
-		(at 159.566 74.168 180)
+		(at 159.439 74.93 180)
 		(descr "JST XH series connector, B6B-XH-A (http://www.jst-mfg.com/product/pdf/eng/eXH.pdf), generated with kicad-footprint-generator")
 		(tags "connector JST XH vertical")
@@
 	(footprint "Connector_JST:JST_XH_B3B-XH-A_1x03_P2.50mm_Vertical"
 		(layer "F.Cu")
-		(at 170.862 74.168 180)
+		(at 170.735 74.93 180)
 		(descr "JST XH series connector, B3B-XH-A (http://www.jst-mfg.com/product/pdf/eng/eXH.pdf), generated with kicad-footprint-generator")
 		(tags "connector JST XH vertical")
@@
 	(footprint "Connector_JST:JST_XH_B2B-XH-A_1x02_P2.50mm_Vertical"
 		(layer "F.Cu")
-		(at 104.14 107.696 -90)
+		(at 105.156 107.696 -90)
 		(descr "JST XH series connector, B2B-XH-A (http://www.jst-mfg.com/product/pdf/eng/eXH.pdf), generated with kicad-footprint-generator")
 		(tags "connector JST XH vertical")
@@
 	(footprint "Connector_JST:JST_XH_B2B-XH-A_1x02_P2.50mm_Vertical"
 		(layer "F.Cu")
-		(at 104.14 99.06 -90)
+		(at 105.156 98.806 -90)
 		(descr "JST XH series connector, B2B-XH-A (http://www.jst-mfg.com/product/pdf/eng/eXH.pdf), generated with kicad-footprint-generator")
 		(tags "connector JST XH vertical")
@@
 	(footprint "Connector_JST:JST_XH_B3B-XH-A_1x03_P2.50mm_Vertical"
 		(layer "F.Cu")
-		(at 129.714 74.168 180)
+		(at 129.587 74.93 180)
 		(descr "JST XH series connector, B3B-XH-A (http://www.jst-mfg.com/product/pdf/eng/eXH.pdf), generated with kicad-footprint-generator")
 		(tags "connector JST XH vertical")
@@
 		(layer "Edge.Cuts")
 	)
-	(segment
-		(start 104.14 101.56)
-		(end 103.93957 101.56)
-		(width 1)
-		(layer "F.Cu")
-		(net 2)
-	)
-	(segment
-		(start 104.08099 110.196)
-		(end 104.14 110.196)
-		(width 0.8)
-		(layer "F.Cu")
-		(net 3)
-	)
-	(segment
-		(start 103.592 110.196)
-		(end 104.14 110.196)
-		(width 0.8)
-		(layer "F.Cu")
-		(net 3)
-	)
-	(segment
-		(start 161.808943 116.402)
-		(end 171.266 116.402)
-		(width 0.2)
-		(layer "F.Cu")
-		(net 17)
-	)
-	(segment
-		(start 161.106 118.099057)
-		(end 161.106 117.104943)
-		(width 0.2)
-		(layer "F.Cu")
-		(net 17)
-	)
-	(segment
-		(start 161.106 117.104943)
-		(end 161.808943 116.402)
-		(width 0.2)
-		(layer "F.Cu")
-		(net 17)
-	)
-	(segment
-		(start 171.266 116.402)
-		(end 172.466 117.602)
-		(width 0.2)
-		(layer "F.Cu")
-		(net 17)
-	)
-	(segment
-		(start 181.958 75.09)
-		(end 181.958 74.168)
-		(width 0.2)
-		(layer "F.Cu")
-		(net 25)
-	)
-	(segment
-		(start 169.926 92.202)
-		(end 171.126 91.002)
-		(width 0.2)
-		(layer "F.Cu")
-		(net 26)
-	)
-	(segment
-		(start 162.052 91.948)
-		(end 162.306 92.202)
-		(width 0.2)
-		(layer "F.Cu")
-		(net 27)
-	)
-	(segment
-		(start 120.142 75.692)
-		(end 118.618 74.168)
-		(width 0.2)
-		(layer "F.Cu")
-		(net 28)
-	)
-	(zone
-		(net 1)
-		(net_name "GND")
-		(layer "B.Cu")
-		(hatch edge 0.5)
-		(connect_pads
-			(clearance 0.5)
-		)
-		(min_thickness 0.25)
-		(filled_areas_thickness no)
-		(fill yes
-			(thermal_gap 0.5)
-			(thermal_bridge_width 0.5)
-		)
-		(polygon
-			(pts
-				(xy 99.822 69.85) (xy 99.822 140.208) (xy 200.152 140.208) (xy 200.152 69.85)
-			)
-		)
-	)
 	(embedded_fonts no)

Commit message: pcb: complete routed board
Routing:
- net +3.3V: track 0.00 -> 211.6 mm
- net +5V: track 0.00 -> 99.8 mm
- net /L_RPWM: track 0.00 -> 58.2 mm
- net /PROX_F_LV: track 0.00 -> 47.5 mm
- net /PROX_R_LV: track 0.00 -> 47.3 mm
- net /PROX_L_LV: track 0.00 -> 47.3 mm
- net /L_LPWM: track 0.00 -> 42.0 mm
- net /L_REN: track 0.00 -> 41.8 mm
- net /L_LEN: track 0.00 -> 39.2 mm
- net /GYRO_SCL: track 0.00 -> 36.0 mm
- net /LINE_L: track 0.00 -> 34.8 mm
- net /GYRO_SDA: track 0.00 -> 31.1 mm
- net /LINE_B: track 0.00 -> 29.8 mm
- net /PROX_R_HV: track 0.00 -> 29.3 mm
- net /PROX_L_HV: track 0.00 -> 27.8 mm
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- added copper zone on B.Cu, net GND
